File: hardware/XC9500XL_development_board.sch (KiCad schematic (older format))
At the start: 12 parts, among them J1 Conn_01x22_Male, J2 Conn_01x22_Male, J3 Conn_01x07_Male, U1 LM1117-3.3, U2 XC9572XLPC44, X1 CXO_DIP14

Commit message: Adds missing capacitor values
Parts:
- C1, C2, C4, C5, C6: value C -> 100nF
- C3: value C -> 10uF
Changed lines of the file:
@@
 P 7850 2350
 F 0 "C2" H 7965 2396 50  0000 L CNN
-F 1 "C" H 7965 2305 50  0000 L CNN
+F 1 "100nF" H 7965 2305 50  0000 L CNN
 F 2 "" H 7888 2200 50  0001 C CNN
 F 3 "~" H 7850 2350 50  0001 C CNN
@@
 P 4750 1700
 F 0 "C4" H 4865 1746 50  0000 L CNN
-F 1 "C" H 4865 1655 50  0000 L CNN
+F 1 "100nF" H 4865 1655 50  0000 L CNN
 F 2 "" H 4788 1550 50  0001 C CNN
 F 3 "~" H 4750 1700 50  0001 C CNN
@@
 P 5100 1700
 F 0 "C5" H 5215 1746 50  0000 L CNN
-F 1 "C" H 5215 1655 50  0000 L CNN
+F 1 "100nF" H 5215 1655 50  0000 L CNN
 F 2 "" H 5138 1550 50  0001 C CNN
 F 3 "~" H 5100 1700 50  0001 C CNN
@@
 P 5450 1700
 F 0 "C6" H 5565 1746 50  0000 L CNN
-F 1 "C" H 5565 1655 50  0000 L CNN
+F 1 "100nF" H 5565 1655 50  0000 L CNN
 F 2 "" H 5488 1550 50  0001 C CNN
 F 3 "~" H 5450 1700 50  0001 C CNN
@@
 P 8050 3800
 F 0 "C1" H 8165 3846 50  0000 L CNN
-F 1 "C" H 8165 3755 50  0000 L CNN
+F 1 "100nF" H 8165 3755 50  0000 L CNN
 F 2 "" H 8088 3650 50  0001 C CNN
 F 3 "~" H 8050 3800 50  0001 C CNN
@@
 P 8850 2350
 F 0 "C3" H 8965 2396 50  0000 L CNN
-F 1 "C" H 8965 2305 50  0000 L CNN
+F 1 "10uF" H 8965 2305 50  0000 L CNN
 F 2 "" H 8888 2200 50  0001 C CNN
 F 3 "~" H 8850 2350 50  0001 C CNN
